Commit message: added stress field prediction model and trainer

File: sim_data/stress_prediction_data/objects/mustard_bottle/soft_body.urdf (robot description, URDF)
Before this commit: robot banana, 1 links, 0 joints
Links:
- removed link banana
- added link mustard_bottle

File: sim_data/stress_prediction_data/objects/rubiks_cube/soft_body.urdf (robot description, URDF)
Before this commit: robot banana, 1 links, 0 joints
Links:
- removed link banana
- added link rubiks_cube

File: sim_data/stress_prediction_data/objects/strawberry/soft_body.urdf (robot description, URDF)
Before this commit: robot banana, 1 links, 0 joints
Links:
- removed link banana
- added link strawberry
