Commit message: add evaluate_and_vis.py

File: sim_data/stress_prediction_data/franka_description/robots/franka_panda_fem_simple_v4_with_arm.urdf (robot description, URDF)
Before this commit: robot panda, 17 links, 16 joints
Links:
- link panda_hand: geometry collision mesh filename=meshes/visual/hand.obj; visual mesh filename=meshes/visual/hand.obj
- link panda_left_finger_rigid: geometry collision mesh filename=meshes/custom/full_fillet_finger.obj; visual mesh filename=meshes/custom/full_fillet_finger.obj
- link panda_right_finger_rigid: geometry collision mesh filename=meshes/custom/full_fillet_finger.obj; visual mesh filename=meshes/custom/full_fillet_finger.obj
